File: Trigon.sch (KiCad schematic (older format))
At the start: 70 parts, among them J1 TYPE-C-31-M12_13, SW1 SW_Push, SW2 Rotary_Encoder_Switch, U1 ATmega32U4-AU, Y1 16MHz

Commit message: USB hub
Parts:
- added C10, C9: 22pF, Capacitor_SMD:C_0805_2012Metric, symbol Device:C_Small
- added C11: 10uF, Capacitor_SMD:C_0805_2012Metric, symbol Device:CP_Small
- added C12, C13, C14, C17, C18, C8: 0.1uF, Capacitor_SMD:C_0805_2012Metric, symbol Device:C_Small
- added C15, C16: 1uF, Capacitor_SMD:C_0805_2012Metric, symbol Device:C_Small
- added D27: 9V Breakdown, acheron_Components:D_SOD-123_Bidirectional, symbol Device:D_TVS
- added F2: 500mA, Fuse:Fuse_1206_3216Metric, symbol Device:Polyfuse_Small
- added FB1, FB2, FB3: 600R, josh-passives-smt:Ferrite_Bead_0603, symbol Device:Ferrite_Bead_Small
- added J2: TYPE-C-31-M12_13, acheronConnectors:TYPE-C-31-M-12, symbol acheronSymbols:TYPE-C-31-M12_13
- added L1, L2: L_Core_Ferrite, Inductor_SMD:L_1206_3216Metric, symbol Device:L_Core_Ferrite
- added MH1, MH2, MH3, MH4: Mount-M2, random-keyboard-parts:Generic-Mounthole, symbol Connector_Generic:Conn_01x01
- added R10: 650R, Resistor_SMD:R_0805_2012Metric, symbol Device:R_Small
- added R7, R8: 100k, Resistor_SMD:R_0805_2012Metric, symbol Device:R_Small
- added R9: 10k, Resistor_SMD:R_0805_2012Metric, symbol Device:R_Small
- added RN1: R_Pack04, Resistor_SMD:R_Array_Convex_4x0603, symbol Device:R_Pack04
- added U2, U4: TPD4E05U06DQAR, Package_SON:USON-10_2.5x1.0mm_P0.5mm, symbol acheronSymbols:TPD4E05U06DQAR
- added U3: CY7C65632-28LTXCT, Package_DFN_QFN:QFN-28-1EP_5x5mm_P0.5mm_EP3.35x3.35mm_ThermalVias, symbol josh-ic:CY7C65632-28LTXCT
- added Y2: 12MHz, Crystal:Crystal_SMD_3225-4Pin_3.2x2.5mm, symbol Device:Crystal_GND24_Small
Connections:
- net labels added: +3.3V, +3.3VA, D1A_D+, D1A_D-, D1B_D+, D1B_D-, D1_D+, D1_D-, D2_D+, D2_D-, D3_D+, D3_D-, DA+, DA-, DB+, DB-, DN, DP, GNDPWR, VBUS, VREG_3V3, nOVR_1, nOVR_2, nOVR_3, nOVR_4
- net labels removed: D+, D-, VCC
- wire segments 149 -> 282
- no-connect marks 0 -> 21
Other:
- note added: "(to 32u4 & keyboard matrix)"
- note added: "(to external usb device)"
- note added: "(to internal usb device)"
- moved on the sheet: C1, C2, C3, C4, C5, C6, C7, D1, D10, D11, D12, D13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

Commit message: usb hub pcb layout
Parts:
- removed RN1: R_Pack04, Resistor_SMD:R_Array_Convex_4x0603, symbol Device:R_Pack04
- added D28: 9V Breakdown, acheron_Components:D_SOD-123_Bidirectional, symbol Device:D_TVS
- added R11, R12, R13, R14: 10k, Resistor_SMD:R_0805_2012Metric, symbol Device:R_Small
- J2: footprint acheronConnectors:TYPE-C-31-M-12 -> acheron_Connectors:TYPE-C-31-M-12
Connections:
- wire segments 282 -> 286
Other:
- note added: "C11 close to Pin 28"
- note added: "USB hub"
- note added: "downstream usb connector + esd protection\n"
- note added: "keyboard matrix\n"
- note added: "keyboard microcontroller\n"
- note added: "upstream usb + esd protection\n"
- moved on the sheet: C1, C10, C2, C3, C4, C5, C6, C7, C8, C9, D27, F1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

Commit message: changes to fuse values per joshajohnson
Parts:
- D27, D28: value 9V Breakdown -> 6V Breakdown
- F2: value 500mA -> 200mA
Changed lines of the file:
@@
 	2300 2850 2450 2850
-$Comp
-L Device:Crystal_GND24_Small Y1
-U 1 1 5F1152C0
-P 1750 2350
-F 0 "Y1" V 1704 2494 50  0000 L CNN
-F 1 "16MHz" V 1795 2494 50  0000 L CNN
-F 2 "Crystal:Crystal_SMD_3225-4Pin_3.2x2.5mm" H 1750 2350 50  0001 C CNN
-F 3 "~" H 1750 2350 50  0001 C CNN
-	1    1750 2350
-	0    1    1    0
-$EndComp
-Wire Wire Line
-	2700 2250 2450 2250
-Wire Wire Line
-	2700 2450 2450 2450
 $Comp
 L Device:C_Small C2
@@
 	1    0    0    -1
 $EndComp
-Connection ~ 2450 2250
 Wire Wire Line
 	2450 2250 1750 2250
-Connection ~ 2450 2450
 Wire Wire Line
 	2450 2450 1750 2450
@@
 Wire Wire Line
 	2400 7250 2400 7350
-$Comp
-L Device:D_TVS D27
-U 1 1 5F53CCD5
-P 4000 7600
-F 0 "D27" V 3954 7679 50  0000 L CNN
-F 1 "9V Breakdown" V 4045 7679 50  0000 L CNN
-F 2 "acheron_Components:D_SOD-123_Bidirectional" H 4000 7600 50  0001 C CNN
-F 3 "~" H 4000 7600 50  0001 C CNN
-	1    4000 7600
-	0    1    1    0
-$EndComp
 Wire Wire Line
 	4000 7250 4000 7450
@@
 P 19400 7950
 F 0 "F2" V 19195 7950 50  0000 C CNN
-F 1 "500mA" V 19286 7950 50  0000 C CNN
+F 1 "200mA" V 19286 7950 50  0000 C CNN
 F 2 "Fuse:Fuse_1206_3216Metric" H 19450 7750 50  0001 L CNN
 F 3 "~" H 19400 7950 50  0001 C CNN
@@
 P 19750 8200
 F 0 "D28" V 19704 8279 50  0000 L CNN
-F 1 "9V Breakdown" V 19795 8279 50  0000 L CNN
+F 1 "6V Breakdown" V 19795 8279 50  0000 L CNN
 F 2 "acheron_Components:D_SOD-123_Bidirectional" H 19750 8200 50  0001 C CNN
 F 3 "~" H 19750 8200 50  0001 C CNN
@@
 Text Notes 16900 7350 0    157  ~ 0
 downstream usb connector + esd protection\n
+$Comp
+L Device:Crystal_GND24_Small Y1
+U 1 1 5F1152C0
+P 1750 2350
+F 0 "Y1" V 1704 2494 50  0000 L CNN
+F 1 "16MHz" V 1795 2494 50  0000 L CNN
+F 2 "Crystal:Crystal_SMD_3225-4Pin_3.2x2.5mm" H 1750 2350 50  0001 C CNN
+F 3 "~" H 1750 2350 50  0001 C CNN
+	1    1750 2350
+	0    1    1    0
+$EndComp
+$Comp
+L Device:D_TVS D27
+U 1 1 5F53CCD5
+P 4000 7600
+F 0 "D27" V 3954 7679 50  0000 L CNN
+F 1 "6V Breakdown" V 4045 7679 50  0000 L CNN
+F 2 "acheron_Components:D_SOD-123_Bidirectional" H 4000 7600 50  0001 C CNN
+F 3 "~" H 4000 7600 50  0001 C CNN
+	1    4000 7600
+	0    1    1    0
+$EndComp
 $EndSCHEMATC

Commit message: More compact layout
Parts:
- C1, C10, C2, C9: footprint Capacitor_SMD:C_0805_2012Metric -> Capacitor_SMD:C_0603_1608Metric; Manufacturer Part # (none) -> CL21C220JBANNNC
- C11, C7: footprint Capacitor_SMD:C_0805_2012Metric -> Capacitor_SMD:C_0603_1608Metric; Manufacturer Part # (none) -> CL21A106KAYNNNE
- C12, C13, C14, C17, C18, C4, C5, C6, C8: footprint Capacitor_SMD:C_0805_2012Metric -> Capacitor_SMD:C_0603_1608Metric; Manufacturer Part # (none) -> CC0805KRX7R9BB104
- C15, C16, C3: footprint Capacitor_SMD:C_0805_2012Metric -> Capacitor_SMD:C_0603_1608Metric; Manufacturer Part # (none) -> CL21B105KBFNNNE
- D1, D10, D11, D12, D13, D14, D15, D16, D17, D18, D19, D2, D20, D21, D22, D23, D24, D25, D26, D3, D4, D5, D6, D7, D8, D9: Manufacturer Part # (none) -> 1N4148W
- D27, D28: Manufacturer Part # (none) -> SMF6.0CA
- F1: Manufacturer Part # (none) -> 1206L050YR
- F2: Manufacturer Part # (none) -> 1206L020YR
- FB1, FB2, FB3: Manufacturer Part # (none) -> BLM18AG601SN1D
- J1, J2: Manufacturer Part # (none) -> TYPE-C-31-M-12
- L1, L2: value L_Core_Ferrite -> 60R@100MHz; Manufacturer Part # (none) -> MLB3216-600P4A(f)
- R1, R2: footprint Resistor_SMD:R_0805_2012Metric -> Resistor_SMD:R_0603_1608Metric; Manufacturer Part # (none) -> 0603WAF220JT5E
- R10: footprint Resistor_SMD:R_0805_2012Metric -> Resistor_SMD:R_0603_1608Metric; Manufacturer Part # (none) -> 0603WAF6500T5E
- R11, R12, R13, R14, R3, R6, R9: footprint Resistor_SMD:R_0805_2012Metric -> Resistor_SMD:R_0603_1608Metric; Manufacturer Part # (none) -> 0603WAF1002T5E
- R4, R5: footprint Resistor_SMD:R_0805_2012Metric -> Resistor_SMD:R_0603_1608Metric; Manufacturer Part # (none) -> 0603WAF5101T5E
- R7, R8: footprint Resistor_SMD:R_0805_2012Metric -> Resistor_SMD:R_0603_1608Metric; Manufacturer Part # (none) -> 0603WAF1003T5E
- SW1: Manufacturer Part # (none) -> TS-1186D-C-A
- U1: Manufacturer Part # (none) -> ATMEGA32U4-AU
- U3: Manufacturer Part # (none) -> CY7C65632-28LTXCT
- Y1: Manufacturer Part # (none) -> X322516MLB4SI
- Y2: Manufacturer Part # (none) -> X322512MOB4SI
Connections:
- net GNDPWR: now also MH1.1 (Pin_1), MH3.1 (Pin_1), MH4.1 (Pin_1)

Commit message: incorporating josh's feedback
Parts:
- removed L1, L2: 60R@100MHz, Inductor_SMD:L_1206_3216Metric, symbol Device:L_Core_Ferrite
- removed U2, U4: TPD4E05U06DQAR, Package_SON:USON-10_2.5x1.0mm_P0.5mm, symbol acheronSymbols:TPD4E05U06DQAR
- added C19, C20, C21: 0.1uF, Capacitor_SMD:C_0603_1608Metric, symbol Device:C_Small
- added FB4: 600R, josh-passives-smt:Ferrite_Bead_0603, symbol Device:Ferrite_Bead_Small
- added R15, R16: 100k, Resistor_SMD:R_0603_1608Metric, symbol Device:R_Small
- added U2, U4: USBLC6-2SC6, Package_TO_SOT_SMD:SOT-23-6, symbol Power_Protection:USBLC6-2SC6
Connections:
- net +3V3: now also C8.1, FB1.2; no longer FB1.1, U3.21 (VCC_D)
- net +5V: now also U1.7 (VBUS), FB4.1; no longer D27.1 (A1), F1.1
- net GND: now also D27.2 (A2), D28.2 (A2), J1.A1 (GND), J1.B1 (GND), J2.A1 (GND), J2.B1 (GND), MH1.1 (Pin_1), MH2.1 (Pin_1), MH3.1 (Pin_1), MH4.1 (Pin_1), R4.1, R5.1, C19.2, C20.2, C21.2, R15.2, R16.2, U2.2 (GND), U4.2 (GND)
- net VBUS: now also F1.2, J1.A4 (VBUS), J1.B4 (VBUS), C21.1, U2.5 (VBUS); no longer U1.7 (VBUS)
- net at C18.1, F2.2, J2.A4 (VBUS)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: now also U4.5 (VBUS)
- net D1A_D+ renamed D1_DP
- net D1_DP: now also U4.3 (IO2); no longer U3.4 (D1_D+)
- net D1A_D- renamed D1_DN
- net D1_DN: now also U4.1 (IO1); no longer U3.3 (D1_D-)
- net DA+ renamed UP_DP
- net UP_DP: now also U2.3 (IO2); no longer U3.2 (UP_D+)
- net DA- renamed UP_DN
- net UP_DN: now also U2.1 (IO1); no longer U3.1 (UP_D-)
- removed net GNDPWR: D27.2 (A2), D28.2 (A2), J1.A1 (GND), J1.B1 (GND), J1.S (SHIELD), J2.A1 (GND), J2.B1 (GND), J2.S (SHIELD), MH1.1 (Pin_1), MH2.1 (Pin_1), MH3.1 (Pin_1), MH4.1 (Pin_1), R4.1, R5.1
- new net: C19.1, J1.S (SHIELD), R15.1
- new net: D27.1 (A1), F1.1, FB4.2
- new net: C20.1, J2.S (SHIELD), R16.1
- new net: FB1.1, U3.21 (VCC_D)
- new net D1_D+: U3.4 (D1_D+), U4.4 (IO2)
- new net D1_D-: U3.3 (D1_D-), U4.6 (IO1)
- new net UP_D+: U2.4 (IO2), U3.2 (UP_D+)
- new net UP_D-: U2.6 (IO1), U3.1 (UP_D-)
Other:
- moved on the sheet: FB1

Commit message: next round of feedback from josh
Parts:
- removed D27, D28: 6V Breakdown, acheron_Components:D_SOD-123_Bidirectional, symbol Device:D_TVS
- added J?: Conn_01x05, symbol Connector_Generic:Conn_01x05
Connections:
- net +5V: now also J?.3 (Pin_3)
- net D2_D+: now also J?.1 (Pin_1)
- net D2_D-: now also J?.2 (Pin_2)
- net GND: now also J?.5 (Pin_5)
- no-connect marks 21 -> 22
Other:
- moved on the sheet: C18, C20, F2, FB3, J2, R16, U4

Commit message: - Introduced JST connector - Made all D+/D- 14mm thick (max thickness that was easy to deal with) - Added logo / decoration / version #
Parts:
- added H1: Logo, Trigon:wiggle, symbol Mechanical:MountingHole
- J3: renamed from J?; footprint (none) -> Connector_JST:JST_SH_SM05B-SRSS-TB_1x05-1MP_P1.00mm_Horizontal
- SW1: Manufacturer Part # TS-1186D-C-A -> TS-1187A-B-A-B
- SW2: footprint Keebio-Parts:RotaryEncoder_Alps_EC11E-Switch_Vertical_H20mm -> Rotary_Encoder:RotaryEncoder_Alps_EC11E-Switch_Vertical_H20mm
Connections:
- net D2_D+: now also U3.16 (D4_D+); no longer U3.7 (D2_D+)
- net D2_D-: now also U3.15 (D4_D-); no longer U3.6 (D2_D-)
Changed lines of the file:
@@
 F 0 "SW2" H 21350 3233 50  0000 C CNN
 F 1 "Rotary_Encoder_Switch" H 21350 3324 50  0000 C CNN
-F 2 "Keebio-Parts:RotaryEncoder_Alps_EC11E-Switch_Vertical_H20mm" H 21200 3760 50  0001 C CNN
+F 2 "Rotary_Encoder:RotaryEncoder_Alps_EC11E-Switch_Vertical_H20mm" H 21200 3760 50  0001 C CNN
 F 3 "~" H 21350 3860 50  0001 C CNN
 	1    21350 3600
@@
 F 2 "random-keyboard-parts:SKQG-1155865" H 1950 1800 50  0001 C CNN
 F 3 "~" H 1950 1800 50  0001 C CNN
-F 4 "TS-1186D-C-A" H 1950 1600 50  0001 C CNN "Manufacturer Part #"
+F 4 "TS-1187A-B-A-B" H 1950 1600 50  0001 C CNN "Manufacturer Part #"
 	1    1950 1600
 	1    0    0    -1
@@
 Text GLabel 11850 9450 2    50   Input ~ 0
 D1_D+
-Text GLabel 11850 9750 2    50   Input ~ 0
+Text GLabel 11850 10550 2    50   Input ~ 0
 D2_D-
-NoConn ~ 11850 10550
-NoConn ~ 11850 10650
 $Comp
 L power:GND #PWR0129
@@
 Text GLabel 11850 9550 2    50   Input ~ 0
 nOVR_1
-Text GLabel 11850 9850 2    50   Input ~ 0
+Text GLabel 11850 10650 2    50   Input ~ 0
 D2_D+
 Text GLabel 11850 9950 2    50   Input ~ 0
@@
 	20150 7150 20600 7150
 $Comp
-L Connector_Generic:Conn_01x05 J?
+L Connector_Generic:Conn_01x05 J3
 U 1 1 5F445C4B
 P 19650 12900
-F 0 "J?" H 19730 12942 50  0000 L CNN
+F 0 "J3" H 19730 12942 50  0000 L CNN
 F 1 "Conn_01x05" H 19730 12851 50  0000 L CNN
-F 2 "" H 19650 12900 50  0001 C CNN
+F 2 "Connector_JST:JST_SH_SM05B-SRSS-TB_1x05-1MP_P1.00mm_Horizontal" H 19650 12900 50  0001 C CNN
 F 3 "~" H 19650 12900 50  0001 C CNN
 	1    19650 12900
@@
 $EndComp
 $Comp
-L power:+5V #PWR?
+L power:+5V #PWR0125
 U 1 1 5F448257
 P 18850 12900
-F 0 "#PWR?" H 18850 12750 50  0001 C CNN
+F 0 "#PWR0125" H 18850 12750 50  0001 C CNN
 F 1 "+5V" H 18865 13073 50  0000 C CNN
 F 2 "" H 18850 12900 50  0001 C CNN
@@
 $EndComp
 $Comp
-L power:GND #PWR?
+L power:GND #PWR0142
 U 1 1 5F449573
 P 19150 13350
-F 0 "#PWR?" H 19150 13100 50  0001 C CNN
+F 0 "#PWR0142" H 19150 13100 50  0001 C CNN
 F 1 "GND" H 19155 13177 50  0000 C CNN
 F 2 "" H 19150 13350 50  0001 C CNN
@@
 	19450 12900 18850 12900
 NoConn ~ 19450 13000
+NoConn ~ 11850 9750
+NoConn ~ 11850 9850
+$Comp
+L Mechanical:MountingHole H1
+U 1 1 5F80E537
+P 1450 14300
+F 0 "H1" H 1550 14346 50  0000 L CNN
+F 1 "Logo" H 1550 14255 50  0000 L CNN
+F 2 "Trigon:wiggle" H 1450 14300 50  0001 C CNN
+F 3 "~" H 1450 14300 50  0001 C CNN
+	1    1450 14300
+	1    0    0    -1
+$EndComp
 $EndSCHEMATC
