File: Hardware/Trigon.sch (KiCad schematic (older format))
At the start: 110 parts, among them J1 TYPE-C-31-M12_13, J2 TYPE-C-31-M12_13, J3 Conn_01x05, SW1 SW_Push, SW2 Rotary_Encoder_Switch, U1 ATmega32U4-AU, U2 USBLC6-2SC6, U3 CY7C65632-28LTXCT, U4 USBLC6-2SC6, Y1 16MHz, Y2 12MHz

Commit message: checkpoint
Parts:
- MH1, MH2, MH3, MH4: footprint random-keyboard-parts:Generic-Mounthole -> CustomMounting:MountingHole_3.2mm_M3_Pad_v2
Connections:
- net COL0: now also U1.30 (PB6); no longer U1.25 (PD4)
- net COL1: now also U1.29 (PB5); no longer U1.26 (PD6)
- net COL3: now also U1.27 (PD7); no longer U1.29 (PB5)
- net COL4: no longer MX5.1 (COL)
- net COL5: now also U1.8 (PB0); no longer SW2.S2, U1.32 (PC7)
- net COL6: now also SW2.S1, U1.12 (PB7); no longer U1.22 (PD5)
- net ENC1A: now also SW2.A, U1.21 (PD3); no longer SW2.B, U1.36 (PF7)
- net ENC1B: now also SW2.B, U1.22 (PD5); no longer SW2.A, U1.37 (PF6)
- net ROW0: now also U1.38 (PF5); no longer D5.1 (K), D6.1 (K), D7.1 (K), U1.12 (PB7)
- net ROW1: no longer D13.1 (K)
- net ROW2: no longer D26.1 (K)
- net ROW3: now also U1.26 (PD6); no longer U1.30 (PB6)
- net ROW4: now also U1.25 (PD4); no longer U1.27 (PD7)
- net ROW0.5: now reaches U1.10 (PB2)
- net ROW0.5: now also D5.1 (K), D6.1 (K), D7.1 (K)
- net ROW1.5: now reaches U1.11 (PB3)
- net ROW1.5: now also D13.1 (K), D26.1 (K)
- net COL3.5: now reaches U1.9 (PB1)
- net COL3.5: now also MX5.1 (COL)
- net at D26.2 (A): now also SW2.S2; no longer SW2.S1
- no-connect marks 23 -> 19
Other:
- moved on the sheet: D26, SW2
Changed lines of the file:
@@
 	19300 3550 19300 4350
 Wire Wire Line
-	20000 1900 20000 2700
-Connection ~ 20000 2700
-Wire Wire Line
 	20000 2700 20000 3550
-Wire Wire Line
-	20750 1900 20750 2700
 Wire Wire Line
 	16600 2300 16950 2300
@@
 Wire Wire Line
 	17650 2300 18300 2300
-Connection ~ 18300 2300
-Wire Wire Line
-	18300 2300 19000 2300
-Connection ~ 19000 2300
-Wire Wire Line
-	19000 2300 19700 2300
-Connection ~ 19700 2300
 Wire Wire Line
 	19700 2300 20450 2300
@@
 Wire Wire Line
 	19000 3100 19700 3100
-Connection ~ 19700 3100
-Wire Wire Line
-	19700 3100 20450 3100
 Wire Wire Line
 	16600 3950 16950 3950
@@
 Connection ~ 19300 1900
 Wire Wire Line
-	20000 1900 20000 1500
-Connection ~ 20000 1900
-Wire Wire Line
 	20750 1900 20750 1500
-Connection ~ 20750 1900
 Wire Wire Line
 	21550 1900 21550 1500
@@
 Text GLabel 19300 1500 1    50   Input ~ 0
 COL3
-Text GLabel 20000 1500 1    50   Input ~ 0
-COL4
 Text GLabel 20750 1500 1    50   Input ~ 0
 COL5
@@
 ROW4
 $Comp
-L MCU_Microchip_ATmega:ATmega32U4-AU U1
-U 1 1 5F0AE892
-P 3050 3550
-F 0 "U1" H 3050 1661 50  0000 C CNN
-F 1 "ATmega32U4-AU" H 3050 1570 50  0000 C CNN
-F 2 "Package_QFP:TQFP-44_10x10mm_P0.8mm" H 3050 3550 50  0001 C CIN
-F 3 "http://ww1.microchip.com/downloads/en/DeviceDoc/Atmel-7766-8-bit-AVR-ATmega16U4-32U4_Datasheet.pdf" H 3050 3550 50  0001 C CNN
-F 4 "ATMEGA32U4-AU" H 3050 3550 50  0001 C CNN "Manufacturer Part #"
-	1    3050 3550
-	1    0    0    -1
-$EndComp
-$Comp
 L Device:Rotary_Encoder_Switch SW2
 U 1 1 5F0AFDB5
-P 21350 3600
-F 0 "SW2" H 21350 3233 50  0000 C CNN
-F 1 "Rotary_Encoder_Switch" H 21350 3324 50  0000 C CNN
-F 2 "Rotary_Encoder:RotaryEncoder_Alps_EC11E-Switch_Vertical_H20mm" H 21200 3760 50  0001 C CNN
-F 3 "~" H 21350 3860 50  0001 C CNN
-	1    21350 3600
-	-1   0    0    1
+P 21700 3000
+F 0 "SW2" H 21700 2633 50  0000 C CNN
+F 1 "Rotary_Encoder_Switch" H 21700 2724 50  0000 C CNN
+F 2 "Rotary_Encoder:RotaryEncoder_Alps_EC11E-Switch_Vertical_H20mm" H 21550 3160 50  0001 C CNN
+F 3 "~" H 21700 3260 50  0001 C CNN
+	1    21700 3000
+	-1   0    0    -1
 $EndComp
 $Comp
 L Device:D_Small D26
 U 1 1 5F0B44C0
-P 20800 3700
-F 0 "D26" V 20846 3632 50  0000 R CNN
-F 1 "D_Small" V 20755 3632 50  0000 R CNN
-F 2 "Diode_SMD:D_SOD-123" V 20800 3700 50  0001 C CNN
-F 3 "~" V 20800 3700 50  0001 C CNN
-F 4 "1N4148W" H 20800 3700 50  0001 C CNN "Manufacturer Part #"
-	1    20800 3700
-	1    0    0    -1
-$EndComp
-Wire Wire Line
-	21050 3700 20900 3700
-Wire Wire Line
-	19700 3950 20700 3950
-Wire Wire Line
-	20700 3950 20700 3700
-Connection ~ 19700 3950
+P 21150 3100
+F 0 "D26" V 21196 3032 50  0000 R CNN
+F 1 "D_Small" V 21105 3032 50  0000 R CNN
+F 2 "Diode_SMD:D_SOD-123" V 21150 3100 50  0001 C CNN
+F 3 "~" V 21150 3100 50  0001 C CNN
+F 4 "1N4148W" H 21150 3100 50  0001 C CNN "Manufacturer Part #"
+	1    21150 3100
+	1    0    0    -1
+$EndComp
+Wire Wire Line
+	21400 3100 21250 3100
 $Comp
 L power:GND #PWR0101
 U 1 1 5F0BA8A5
-P 21950 3600
-F 0 "#PWR0101" H 21950 3350 50  0001 C CNN
-F 1 "GND" V 21955 3472 50  0000 R CNN
-F 2 "" H 21950 3600 50  0001 C CNN
-F 3 "" H 21950 3600 50  0001 C CNN
-	1    21950 3600
+P 22300 3000
+F 0 "#PWR0101" H 22300 2750 50  0001 C CNN
+F 1 "GND" V 22305 2872 50  0000 R CNN
+F 2 "" H 22300 3000 50  0001 C CNN
+F 3 "" H 22300 3000 50  0001 C CNN
+	1    22300 3000
 	0    -1   -1   0
 $EndComp
 Wire Wire Line
-	21650 3600 21950 3600
-Text GLabel 21650 3500 2    50   Input ~ 0
+	22000 3000 22300 3000
+Text GLabel 22000 2900 2    50   Input ~ 0
 ENC1A
-Text GLabel 21650 3700 2    50   Input ~ 0
+Text GLabel 22000 3100 2    50   Input ~ 0
 ENC1B
 $Comp
@@
 Wire Wire Line
 	2950 1550 2950 1750
-Wire Wire Line
-	2950 1750 3050 1750
-Connection ~ 2950 1750
-Connection ~ 3050 1750
-Wire Wire Line
-	3050 1750 3150 1750
 $Comp
 L power:GND #PWR0103
@@
 $EndComp
 Wire Wire Line
-	3050 5350 2950 5350
-Wire Wire Line
 	2550 5350 2550 5450
-Connection ~ 2950 5350
-Wire Wire Line
-	2950 5350 2550 5350
 $Comp
 L Device:R_Small R6
@@
 	0    1    1    0
 $EndComp
-Wire Wire Line
-	21050 3500 20750 3500
-Wire Wire Line
-	20750 3500 20750 2700
-Connection ~ 20750 2700
-Text GLabel 3650 3650 2    50   Input ~ 0
+Text GLabel 3650 2650 2    50   Input ~ 0
 COL0
-Text GLabel 3650 3850 2    50   Input ~ 0
+Text GLabel 3650 2550 2    50   Input ~ 0
 COL1
 Text GLabel 3650 2450 2    50   Input ~ 0
 COL2
-Text GLabel 3650 2550 2    50   Input ~ 0
+Text GLabel 3650 3950 2    50   Input ~ 0
 COL3
 Text GLabel 3650 2950 2    50   Input ~ 0
 COL4
-Text GLabel 3650 3050 2    50   Input ~ 0
+Text GLabel 3650 2050 2    50   Input ~ 0
 COL5
-Text GLabel 3650 3750 2    50   Input ~ 0
+Text GLabel 3650 2750 2    50   Input ~ 0
 COL6
-Text GLabel 3650 2750 2    50   Input ~ 0
-ROW0
-Text GLabel 3650 3950 2    50   Input ~ 0
+Text GLabel 3650 3650 2    50   Input ~ 0
 ROW4
-Text GLabel 3650 2650 2    50   Input ~ 0
+Text GLabel 3650 3850 2    50   Input ~ 0
 ROW3
 Text GLabel 3650 4650 2    50   Input ~ 0
@@
 Text GLabel 3650 4450 2    50   Input ~ 0
 ROW1
-Text GLabel 3650 4850 2    50   Input ~ 0
+Text GLabel 3650 3750 2    50   Input ~ 0
 ENC1B
-Text GLabel 3650 4950 2    50   Input ~ 0
+Text GLabel 3650 3550 2    50   Input ~ 0
 ENC1A
 Wire Wire Line
@@
 F 0 "MH1" H 1480 15742 50  0000 L CNN
 F 1 "Mount-M2" H 1480 15651 50  0000 L CNN
-F 2 "random-keyboard-parts:Generic-Mounthole" H 1400 15700 50  0001 C CNN
+F 2 "CustomMounting:MountingHole_3.2mm_M3_Pad_v2" H 1400 15700 50  0001 C CNN
 F 3 "~" H 1400 15700 50  0001 C CNN
 	1    1400 15700
@@
 F 0 "MH2" H 1480 15442 50  0000 L CNN
 F 1 "Mount-M2" H 1480 15351 50  0000 L CNN
-F 2 "random-keyboard-parts:Generic-Mounthole" H 1400 15400 50  0001 C CNN
+F 2 "CustomMounting:MountingHole_3.2mm_M3_Pad_v2" H 1400 15400 50  0001 C CNN
 F 3 "~" H 1400 15400 50  0001 C CNN
 	1    1400 15400
@@
 F 0 "MH3" H 1480 15142 50  0000 L CNN
 F 1 "Mount-M2" H 1480 15051 50  0000 L CNN
-F 2 "random-keyboard-parts:Generic-Mounthole" H 1400 15100 50  0001 C CNN
+F 2 "CustomMounting:MountingHole_3.2mm_M3_Pad_v2" H 1400 15100 50  0001 C CNN
 F 3 "~" H 1400 15100 50  0001 C CNN
 	1    1400 15100
@@
 F 0 "MH4" H 1480 14842 50  0000 L CNN
 F 1 "Mount-M2" H 1480 14751 50  0000 L CNN
-F 2 "random-keyboard-parts:Generic-Mounthole" H 1400 14800 50  0001 C CNN
+F 2 "CustomMounting:MountingHole_3.2mm_M3_Pad_v2" H 1400 14800 50  0001 C CNN
 F 3 "~" H 1400 14800 50  0001 C CNN
 	1    1400 14800
@@
 Wire Notes Line
 	2150 14550 750  14550
-NoConn ~ 3650 2050
-NoConn ~ 3650 2150
-NoConn ~ 3650 2250
-NoConn ~ 3650 2350
 NoConn ~ 3650 3250
 NoConn ~ 3650 3350
 NoConn ~ 3650 3450
-NoConn ~ 3650 3550
 NoConn ~ 3650 4250
 NoConn ~ 3650 4550
-NoConn ~ 3650 4750
 $Comp
 L power:+5V #PWR0123
@@
 	19450 12300 19250 12300
 NoConn ~ 19450 12800
-NoConn ~ 13150 12200
+Wire Wire Line
+	21050 3100 20450 3100
+Wire Wire Line
+	21400 2900 21400 2500
+Wire Wire Line
+	21400 2500 21550 2500
+Wire Wire Line
+	21550 2500 21550 1900
+Connection ~ 21550 1900
+Wire Wire Line
+	2950 5350 2550 5350
+Wire Wire Line
+	3050 5350 2950 5350
+Connection ~ 2950 5350
+Connection ~ 2950 1750
+Wire Wire Line
+	3050 1750 3150 1750
+Wire Wire Line
+	2950 1750 3050 1750
+Connection ~ 3050 1750
+Text GLabel 3650 4750 2    50   Input ~ 0
+ROW0
+Connection ~ 20750 1900
+Wire Wire Line
+	20750 1900 20750 2700
+Text GLabel 20250 2600 1    50   Input ~ 0
+COL4
+Connection ~ 18300 2300
+Wire Wire Line
+	18300 2300 19000 2300
+Wire Wire Line
+	20250 2600 20250 2700
+Wire Wire Line
+	20250 2700 20000 2700
+Connection ~ 20000 2700
+Text GLabel 20000 1550 1    50   Input ~ 0
+COL3.5
+Wire Wire Line
+	20000 1550 20000 1900
+Wire Wire Line
+	19600 1750 19600 2300
+Wire Wire Line
+	19600 2300 19700 2300
+Connection ~ 19700 2300
+Text GLabel 3650 2250 2    50   Input ~ 0
+ROW0.5
+$Comp
+L MCU_Microchip_ATmega:ATmega32U4-AU U1
+U 1 1 5F0AE892
+P 3050 3550
+F 0 "U1" H 3050 1661 50  0000 C CNN
+F 1 "ATmega32U4-AU" H 3050 1570 50  0000 C CNN
+F 2 "Package_QFP:TQFP-44_10x10mm_P0.8mm" H 3050 3550 50  0001 C CIN
+F 3 "http://ww1.microchip.com/downloads/en/DeviceDoc/Atmel-7766-8-bit-AVR-ATmega16U4-32U4_Datasheet.pdf" H 3050 3550 50  0001 C CNN
+F 4 "ATMEGA32U4-AU" H 3050 3550 50  0001 C CNN "Manufacturer Part #"
+	1    3050 3550
+	1    0    0    -1
+$EndComp
+Text GLabel 3650 2150 2    50   Input ~ 0
+COL3.5
+Text GLabel 20450 3350 0    50   Input ~ 0
+ROW1.5
+Wire Wire Line
+	20450 3350 20450 3100
+Connection ~ 20450 3100
+Text GLabel 3650 2350 2    50   Input ~ 0
+ROW1.5
+NoConn ~ 3650 4850
+NoConn ~ 3650 4950
+NoConn ~ 3650 3050
+Text GLabel 19600 1750 1    50   Input ~ 0
+ROW0.5
 $EndSCHEMATC

Commit message: kailh hotswap switches ;now using a fixed acheron
Parts:
- J1, J2: symbol acheronSymbols:TYPE-C-31-M12_13 -> Trigon-rescue:TYPE-C-31-M12_13-acheronSymbols
- MX1, MX10, MX11, MX12, MX13, MX14, MX15, MX16, MX17, MX18, MX19, MX2, MX20, MX21, MX22, MX23, MX24, MX25, MX3, MX4, MX5, MX6, MX7, MX8, MX9: footprint MX_Only:MXOnly-1U-NoLED -> josh-keyboard:Kailh_Hotswap_1U
Connections:
- net COL3.5: no longer MX5.1 (COL)
- net COL4: now also MX5.1 (COL)
Changed lines of the file:
@@
 F 0 "MX1" H 17133 2173 60  0000 C CNN
 F 1 "MX-NoLED" H 17133 2099 20  0000 C CNN
-F 2 "MX_Only:MXOnly-1U-NoLED" H 16475 1925 60  0001 C CNN
+F 2 "josh-keyboard:Kailh_Hotswap_1U" H 16475 1925 60  0001 C CNN
 F 3 "" H 16475 1925 60  0001 C CNN
 	1    17100 1950
@@
 F 0 "MX2" H 17833 2173 60  0000 C CNN
 F 1 "MX-NoLED" H 17833 2099 20  0000 C CNN
-F 2 "MX_Only:MXOnly-1U-NoLED" H 17175 1925 60  0001 C CNN
+F 2 "josh-keyboard:Kailh_Hotswap_1U" H 17175 1925 60  0001 C CNN
 F 3 "" H 17175 1925 60  0001 C CNN
 	1    17800 1950
@@
 F 0 "MX3" H 18483 2173 60  0000 C CNN
 F 1 "MX-NoLED" H 18483 2099 20  0000 C CNN
-F 2 "MX_Only:MXOnly-1U-NoLED" H 17825 1925 60  0001 C CNN
+F 2 "josh-keyboard:Kailh_Hotswap_1U" H 17825 1925 60  0001 C CNN
 F 3 "" H 17825 1925 60  0001 C CNN
 	1    18450 1950
@@
 	18400 2100 18300 2100
 $Comp
-L MX_Alps_Hybrid:MX-NoLED MX4
-U 1 1 5F0712F3
-P 19150 1950
-F 0 "MX4" H 19183 2173 60  0000 C CNN
-F 1 "MX-NoLED" H 19183 2099 20  0000 C CNN
-F 2 "MX_Only:MXOnly-1U-NoLED" H 18525 1925 60  0001 C CNN
-F 3 "" H 18525 1925 60  0001 C CNN
-	1    19150 1950
-	1    0    0    -1
-$EndComp
-$Comp
 L Device:D_Small D4
 U 1 1 5F0712FD
@@
 F 0 "MX5" H 19883 2173 60  0000 C CNN
 F 1 "MX-NoLED" H 19883 2099 20  0000 C CNN
-F 2 "MX_Only:MXOnly-1U-NoLED" H 19225 1925 60  0001 C CNN
+F 2 "josh-keyboard:Kailh_Hotswap_1U" H 19225 1925 60  0001 C CNN
 F 3 "" H 19225 1925 60  0001 C CNN
 	1    19850 1950
@@
 F 0 "MX6" H 20633 2173 60  0000 C CNN
 F 1 "MX-NoLED" H 20633 2099 20  0000 C CNN
-F 2 "MX_Only:MXOnly-1U-NoLED" H 19975 1925 60  0001 C CNN
+F 2 "josh-keyboard:Kailh_Hotswap_1U" H 19975 1925 60  0001 C CNN
 F 3 "" H 19975 1925 60  0001 C CNN
 	1    20600 1950
@@
 F 0 "MX7" H 21433 2173 60  0000 C CNN
 F 1 "MX-NoLED" H 21433 2099 20  0000 C CNN
-F 2 "MX_Only:MXOnly-1U-NoLED" H 20775 1925 60  0001 C CNN
+F 2 "josh-keyboard:Kailh_Hotswap_1U" H 20775 1925 60  0001 C CNN
 F 3 "" H 20775 1925 60  0001 C CNN
 	1    21400 1950
@@
 F 0 "MX8" H 17133 2973 60  0000 C CNN
 F 1 "MX-NoLED" H 17133 2899 20  0000 C CNN
-F 2 "MX_Only:MXOnly-1U-NoLED" H 16475 2725 60  0001 C CNN
+F 2 "josh-keyboard:Kailh_Hotswap_1U" H 16475 2725 60  0001 C CNN
 F 3 "" H 16475 2725 60  0001 C CNN
 	1    17100 2750
@@
 F 0 "MX9" H 17833 2973 60  0000 C CNN
 F 1 "MX-NoLED" H 17833 2899 20  0000 C CNN
-F 2 "MX_Only:MXOnly-1U-NoLED" H 17175 2725 60  0001 C CNN
+F 2 "josh-keyboard:Kailh_Hotswap_1U" H 17175 2725 60  0001 C CNN
 F 3 "" H 17175 2725 60  0001 C CNN
 	1    17800 2750
@@
 F 0 "MX10" H 18483 2973 60  0000 C CNN
 F 1 "MX-NoLED" H 18483 2899 20  0000 C CNN
-F 2 "MX_Only:MXOnly-1U-NoLED" H 17825 2725 60  0001 C CNN
+F 2 "josh-keyboard:Kailh_Hotswap_1U" H 17825 2725 60  0001 C CNN
 F 3 "" H 17825 2725 60  0001 C CNN
 	1    18450 2750
@@
 F 0 "MX11" H 19183 2973 60  0000 C CNN
 F 1 "MX-NoLED" H 19183 2899 20  0000 C CNN
-F 2 "MX_Only:MXOnly-1U-NoLED" H 18525 2725 60  0001 C CNN
+F 2 "josh-keyboard:Kailh_Hotswap_1U" H 18525 2725 60  0001 C CNN
 F 3 "" H 18525 2725 60  0001 C CNN
 	1    19150 2750
@@
 F 0 "MX12" H 19883 2973 60  0000 C CNN
 F 1 "MX-NoLED" H 19883 2899 20  0000 C CNN
-F 2 "MX_Only:MXOnly-1U-NoLED" H 19225 2725 60  0001 C CNN
+F 2 "josh-keyboard:Kailh_Hotswap_1U" H 19225 2725 60  0001 C CNN
 F 3 "" H 19225 2725 60  0001 C CNN
 	1    19850 2750
@@
 F 0 "MX13" H 20633 2973 60  0000 C CNN
 F 1 "MX-NoLED" H 20633 2899 20  0000 C CNN
-F 2 "MX_Only:MXOnly-1U-NoLED" H 19975 2725 60  0001 C CNN
+F 2 "josh-keyboard:Kailh_Hotswap_1U" H 19975 2725 60  0001 C CNN
 F 3 "" H 19975 2725 60  0001 C CNN
 	1    20600 2750
@@
 F 0 "MX14" H 17133 3823 60  0000 C CNN
 F 1 "MX-NoLED" H 17133 3749 20  0000 C CNN
-F 2 "MX_Only:MXOnly-1U-NoLED" H 16475 3575 60  0001 C CNN
+F 2 "josh-keyboard:Kailh_Hotswap_1U" H 16475 3575 60  0001 C CNN
 F 3 "" H 16475 3575 60  0001 C CNN
 	1    17100 3600
@@
 F 0 "MX15" H 17833 3823 60  0000 C CNN
 F 1 "MX-NoLED" H 17833 3749 20  0000 C CNN
-F 2 "MX_Only:MXOnly-1U-NoLED" H 17175 3575 60  0001 C CNN
+F 2 "josh-keyboard:Kailh_Hotswap_1U" H 17175 3575 60  0001 C CNN
 F 3 "" H 17175 3575 60  0001 C CNN
 	1    17800 3600
@@
 F 0 "MX16" H 18483 3823 60  0000 C CNN
 F 1 "MX-NoLED" H 18483 3749 20  0000 C CNN
-F 2 "MX_Only:MXOnly-1U-NoLED" H 17825 3575 60  0001 C CNN
+F 2 "josh-keyboard:Kailh_Hotswap_1U" H 17825 3575 60  0001 C CNN
 F 3 "" H 17825 3575 60  0001 C CNN
 	1    18450 3600
@@
 F 0 "MX17" H 19183 3823 60  0000 C CNN
 F 1 "MX-NoLED" H 19183 3749 20  0000 C CNN
-F 2 "MX_Only:MXOnly-1U-NoLED" H 18525 3575 60  0001 C CNN
+F 2 "josh-keyboard:Kailh_Hotswap_1U" H 18525 3575 60  0001 C CNN
 F 3 "" H 18525 3575 60  0001 C CNN
 	1    19150 3600
@@
 F 0 "MX18" H 19883 3823 60  0000 C CNN
 F 1 "MX-NoLED" H 19883 3749 20  0000 C CNN
-F 2 "MX_Only:MXOnly-1U-NoLED" H 19225 3575 60  0001 C CNN
+F 2 "josh-keyboard:Kailh_Hotswap_1U" H 19225 3575 60  0001 C CNN
 F 3 "" H 19225 3575 60  0001 C CNN
 	1    19850 3600
@@
 F 0 "MX19" H 17133 4623 60  0000 C CNN
 F 1 "MX-NoLED" H 17133 4549 20  0000 C CNN
-F 2 "MX_Only:MXOnly-1U-NoLED" H 16475 4375 60  0001 C CNN
+F 2 "josh-keyboard:Kailh_Hotswap_1U" H 16475 4375 60  0001 C CNN
 F 3 "" H 16475 4375 60  0001 C CNN
 	1    17100 4400
@@
 F 0 "MX20" H 17833 4623 60  0000 C CNN
 F 1 "MX-NoLED" H 17833 4549 20  0000 C CNN
-F 2 "MX_Only:MXOnly-1U-NoLED" H 17175 4375 60  0001 C CNN
+F 2 "josh-keyboard:Kailh_Hotswap_1U" H 17175 4375 60  0001 C CNN
 F 3 "" H 17175 4375 60  0001 C CNN
 	1    17800 4400
@@
 F 0 "MX21" H 18483 4623 60  0000 C CNN
 F 1 "MX-NoLED" H 18483 4549 20  0000 C CNN
-F 2 "MX_Only:MXOnly-1U-NoLED" H 17825 4375 60  0001 C CNN
+F 2 "josh-keyboard:Kailh_Hotswap_1U" H 17825 4375 60  0001 C CNN
 F 3 "" H 17825 4375 60  0001 C CNN
 	1    18450 4400
@@
 F 0 "MX22" H 19183 4623 60  0000 C CNN
 F 1 "MX-NoLED" H 19183 4549 20  0000 C CNN
-F 2 "MX_Only:MXOnly-1U-NoLED" H 18525 4375 60  0001 C CNN
+F 2 "josh-keyboard:Kailh_Hotswap_1U" H 18525 4375 60  0001 C CNN
 F 3 "" H 18525 4375 60  0001 C CNN
 	1    19150 4400
@@
 F 0 "MX23" H 17133 5473 60  0000 C CNN
 F 1 "MX-NoLED" H 17133 5399 20  0000 C CNN
-F 2 "MX_Only:MXOnly-1U-NoLED" H 16475 5225 60  0001 C CNN
+F 2 "josh-keyboard:Kailh_Hotswap_1U" H 16475 5225 60  0001 C CNN
 F 3 "" H 16475 5225 60  0001 C CNN
 	1    17100 5250
@@
 F 0 "MX24" H 17833 5473 60  0000 C CNN
 F 1 "MX-NoLED" H 17833 5399 20  0000 C CNN
-F 2 "MX_Only:MXOnly-1U-NoLED" H 17175 5225 60  0001 C CNN
+F 2 "josh-keyboard:Kailh_Hotswap_1U" H 17175 5225 60  0001 C CNN
 F 3 "" H 17175 5225 60  0001 C CNN
 	1    17800 5250
@@
 F 0 "MX25" H 18483 5473 60  0000 C CNN
 F 1 "MX-NoLED" H 18483 5399 20  0000 C CNN
-F 2 "MX_Only:MXOnly-1U-NoLED" H 17825 5225 60  0001 C CNN
+F 2 "josh-keyboard:Kailh_Hotswap_1U" H 17825 5225 60  0001 C CNN
 F 3 "" H 17825 5225 60  0001 C CNN
 	1    18450 5250
@@
 	18600 4350 18600 5200
 Wire Wire Line
-	19300 1900 19300 2700
-Connection ~ 19300 2700
-Wire Wire Line
 	19300 2700 19300 3550
 Connection ~ 19300 3550
@@
 	18600 1900 18600 1500
 Connection ~ 18600 1900
-Wire Wire Line
-	19300 1900 19300 1500
-Connection ~ 19300 1900
 Wire Wire Line
 	20750 1900 20750 1500
@@
 Connection ~ 2400 7250
 $Comp
-L acheronSymbols:TYPE-C-31-M12_13 J1
+L Trigon-rescue:TYPE-C-31-M12_13-acheronSymbols J1
 U 1 1 5F0D4270
 P 1800 8400
@@
 Connection ~ 18600 9700
 $Comp
-L acheronSymbols:TYPE-C-31-M12_13 J2
+L Trigon-rescue:TYPE-C-31-M12_13-acheronSymbols J2
 U 1 1 5FEBE3CF
 P 18600 8250
@@
 Wire Wire Line
 	20750 1900 20750 2700
-Text GLabel 20250 2600 1    50   Input ~ 0
+Text GLabel 20000 1500 1    50   Input ~ 0
 COL4
 Connection ~ 18300 2300
 Wire Wire Line
 	18300 2300 19000 2300
-Wire Wire Line
-	20250 2600 20250 2700
-Wire Wire Line
-	20250 2700 20000 2700
-Connection ~ 20000 2700
-Text GLabel 20000 1550 1    50   Input ~ 0
-COL3.5
-Wire Wire Line
-	20000 1550 20000 1900
 Wire Wire Line
 	19600 1750 19600 2300
@@
 Text GLabel 19600 1750 1    50   Input ~ 0
 ROW0.5
+Wire Wire Line
+	20000 1500 20000 1900
+Wire Wire Line
+	20000 1900 20000 2700
+Connection ~ 20000 1900
+Connection ~ 20000 2700
+Wire Wire Line
+	19300 1500 19300 1900
+$Comp
+L MX_Alps_Hybrid:MX-NoLED MX4
+U 1 1 5F0712F3
+P 19150 1950
+F 0 "MX4" H 19183 2173 60  0000 C CNN
+F 1 "MX-NoLED" H 19183 2099 20  0000 C CNN
+F 2 "josh-keyboard:Kailh_Hotswap_1U" H 18525 1925 60  0001 C CNN
+F 3 "" H 18525 1925 60  0001 C CNN
+	1    19150 1950
+	1    0    0    -1
+$EndComp
+Wire Wire Line
+	19300 1900 19300 2700
+Connection ~ 19300 1900
+Connection ~ 19300 2700
 $EndSCHEMATC
