File: Hardware/Trigon.kicad_pcb (KiCad board)
At the start: 2 copper layers, 160 x 120 mm, 110 parts, among them J1 TYPE-C-31-M12_13, J2 TYPE-C-31-M12_13, J3 Conn_01x05, SW1 SW_Push, SW2 Rotary_Encoder_Switch, U1 ATmega32U4-AU, U2 USBLC6-2SC6, U3 CY7C65632-28LTXCT, U4 USBLC6-2SC6, Y1 16MHz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

Commit message: lots of changes
Parts:
- moved C19 38.1 mm to (121.3, 18.3)
- moved C21 38.1 mm to (124.4, 22.2)
- moved F1 38.1 mm to (123.6, 24.1)
- moved FB4 38.1 mm to (120.5, 24.9)
- moved J1 38.1 mm to (127.7, 20.6)
- moved R15 38.1 mm to (119.8, 18.2)
- moved R4 38.1 mm to (120.6, 20.6)
- moved R5 38.1 mm to (130.2, 23.4)
- moved U2 38.1 mm to (127.7, 23.8)
Connections:
- net COL3.5 renamed Net-(U1-Pad9)
- net D2_D+ renamed D4_D+
- net D2_D- renamed D4_D-
Routing:
- net +5V: track 224.8 -> 248.1 mm
- net UP_D+: track 20.0 -> 42.0 mm
- net UP_D-: track 20.0 -> 41.0 mm
- net D1_D+: track 58.0 -> 59.9 mm
- net D1_D-: track 57.2 -> 59.0 mm
Other:
- outline, holes or cut-outs redrawn
- board text added: "rev 0.1.2.3"
- board text removed: "rev 0.1.1"

Commit message: preping for pcbway
Parts:
- added H2: Logo, Trigon:back, B.Cu at (92.2, 70.6)
- added H3: Logo, Trigon:backside, F.Cu at (92.1, 72.0)
Routing:
- net UP_D+: track 42.0 -> 44.1 mm
- net GND: track 53.5 -> 51.6 mm, vias 46 -> 48
- net UP_D-: track 41.0 -> 42.8 mm
- net +3.3VA: track 86.9 -> 86.0 mm, vias 3 -> 4
Other:
- outline, holes or cut-outs redrawn
- board text added: "fatto a mano a parigi - nkultra"
- board text added: "rev 0.1.2.4"
- board text removed: "by"
- board text removed: "nkultra"
- board text removed: "rev 0.1.2.3"
- board text removed: "Δkb"
